Commit message: fix: fixed error rostopic of image_raw retrieval
/camera/image_raw --> /${camera_id}/camera/image_raw

File: src/mbot_description/urdf/mbot_with_camera_laser_gazebo_sweep.xacro (robot description, xacro)
@@ -7,4 +7,5 @@
     <xacro:property name="camera_offset_y" value="0" />
     <xacro:property name="camera_offset_z" value="0.10" />
+    <xacro:property name="camera_id" value="camera_center" />
     <xacro:property name="pillar_length" value="0.1" />
     <xacro:property name="pillar_radius" value="0.01" />
@@ -17,7 +18,7 @@
         <origin xyz="${camera_offset_x} ${camera_offset_y} ${camera_offset_z}" rpy="0 0 0" />
         <parent link="base_link"/>
-        <child link="camera_link"/>
+        <child link="${camera_id}_link"/>
     </joint>
-    <xacro:usb_camera prefix="camera"/>
+    <xacro:usb_camera prefix="${camera_id}"/>
     <link name="pillar_link">
         <visual>
